File: MuteBlock.kicad_sch (KiCad schematic)
At the start: 5 parts, among them K3 G5V-2

Commit message: Finished up schematic, before board splitting
Parts:
- JP1, JP13, JP5, JP9: footprint (none) -> Jumper:SolderJumper-2_P1.3mm_Open_RoundedPad1.0x1.5mm
- K3: footprint Relay_THT:Relay_StandexMeder_UMS -> Relay_THT:Relay_DPDT_Omron_G5V-2
Changed lines of the file:
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@@
       (effects (font (size 1.27 1.27)))
     )
-    (property "Footprint" "" (at 110.49 127 0)
+    (property "Footprint" "Jumper:SolderJumper-2_P1.3mm_Open_RoundedPad1.0x1.5mm" (at 110.49 127 0)
       (effects (font (size 1.27 1.27)) hide)
     )
@@
       (effects (font (size 1.27 1.27)))
     )
-    (property "Footprint" "" (at 110.49 133.35 0)
+    (property "Footprint" "Jumper:SolderJumper-2_P1.3mm_Open_RoundedPad1.0x1.5mm" (at 110.49 133.35 0)
       (effects (font (size 1.27 1.27)) hide)
     )
@@
       (effects (font (size 1.27 1.27)))
     )
-    (property "Footprint" "" (at 142.24 127 0)
+    (property "Footprint" "Jumper:SolderJumper-2_P1.3mm_Open_RoundedPad1.0x1.5mm" (at 142.24 127 0)
       (effects (font (size 1.27 1.27)) hide)
     )
@@
       (effects (font (size 1.27 1.27)))
     )
-    (property "Footprint" "Relay_THT:Relay_StandexMeder_UMS" (at 135.89 111.76 0)
+    (property "Footprint" "Relay_THT:Relay_DPDT_Omron_G5V-2" (at 135.89 111.76 0)
       (effects (font (size 1.27 1.27)) (justify left) hide)
     )
@@
       (effects (font (size 1.27 1.27)))
     )
-    (property "Footprint" "" (at 142.24 133.35 0)
+    (property "Footprint" "Jumper:SolderJumper-2_P1.3mm_Open_RoundedPad1.0x1.5mm" (at 142.24 133.35 0)
       (effects (font (size 1.27 1.27)) hide)
     )

Commit message: Changed position of ribbon connectors, added DC
Other:
- company: (none) -> Daniel Machnik Sounddesign und Tontechnik
- title: (none) -> Essigfabrik 2-Way PA Switcher
Changed lines of the file:
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@@
 (kicad_sch (version 20230121) (generator eeschema)
   (paper "A4")
+  (title_block
+    (title "Essigfabrik 2-Way PA Switcher")
+    (date "2023-11-21")
+    (rev "1")
+    (company "Daniel Machnik Sounddesign und Tontechnik")
+  )
   (junction (at 170.18 95.25) (diameter 0) (color 0 0 0 0)
   )
