File: SwitchBlock.kicad_sch (KiCad schematic)
At the start: 1 part, among them K3 G5V-2

Commit message: Finished up schematic, before board splitting
Parts:
- K3: footprint Relay_THT:Relay_StandexMeder_UMS -> Relay_THT:Relay_DPDT_Omron_G5V-2
Changed lines of the file:
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@@
       (effects (font (size 1.27 1.27)))
     )
-    (property "Footprint" "Relay_THT:Relay_StandexMeder_UMS" (at 135.89 102.87 0)
+    (property "Footprint" "Relay_THT:Relay_DPDT_Omron_G5V-2" (at 135.89 102.87 0)
       (effects (font (size 1.27 1.27)) (justify left) hide)
     )

Commit message: Changed position of ribbon connectors, added DC
Other:
- company: (none) -> Daniel Machnik Sounddesign und Tontechnik
- title: (none) -> Essigfabrik 2-Way PA Switcher
Changed lines of the file:
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@@
 (kicad_sch (version 20230121) (generator eeschema)
   (paper "A4")
+  (title_block
+    (title "Essigfabrik 2-Way PA Switcher")
+    (date "2023-11-21")
+    (rev "1")
+    (company "Daniel Machnik Sounddesign und Tontechnik")
+  )
   (wire (pts (xy 114.3 76.2) (xy 127 76.2))
     (stroke (width 0) (type default))
